Commit message: fixed some bugs, added png to rviz, updated readme

File: src/models_pkg/rcCar_assembly/model.urdf (robot description, URDF)
Before this commit: robot automobile, 10 links, 9 joints
Joints:
- joint automobile_joint_leftfront_steer: limit lower=-1.79769e+308 upper=1.79769e+308 effort=-1.0 velocity=-1.0 -> lower=-1.5708 upper=1.5708 effort=1.0 velocity=1.0
- joint automobile_joint_leftrear_rim: limit lower=-1.79769e+308 upper=1.79769e+308 effort=-1.0 velocity=-1.0 -> lower=-1.5708 upper=1.5708 effort=1.0 velocity=1.0
- joint automobile_joint_rightfront_steer: limit lower=-1.79769e+308 upper=1.79769e+308 effort=-1.0 velocity=-1.0 -> lower=-1.5708 upper=1.5708 effort=1.0 velocity=1.0
- joint automobile_joint_rightrear_rim: limit lower=-1.79769e+308 upper=1.79769e+308 effort=-1.0 velocity=-1.0 -> lower=-1.5708 upper=1.5708 effort=1.0 velocity=1.0
